File: design/Millburn_Test_Board/Millburn_Test_Board.kicad_pcb (KiCad board)
At the start: 2 copper layers, 68.6 x 66 mm, 17 parts, among them J1 Conn_01x10, J2 Conn_01x10, J3 Conn_01x10, J4 Conn_01x10, J5 Barrel_Jack_MountingPin

Commit message: Test board: a new revision, with two drawing layers
Re-exported from KiCad. The board keeps its size, its outline and all 42 holes
(36 plated in 9 sizes, 6 non-plated in 6), and the copper is redrawn: front
isolation falls 6262 to 5578 mm of cutting, back 3189 to 2551, with a paste
aperture changing from a 3.6 mm circle to a 4.6 x 2.0 mm rectangle.

Adds F_Courtyard and User_Comments, exported on purpose: they are the first
"Other,..." files in any board here, and they are what showed that such files
were being called Unknown and listed without names.

The golden snapshots cover GridStripConnector, its panelised form and
PogoTest1, so none of them are affected. RealBoards does load this one, and the
suite is green against the new files. A full export plans every program with no
refusals and no gouges.

Co-Authored-By: Claude Opus 5 <noreply@anthropic.com>
Claude-Session: https://claude.ai/code/session_01QyW1VZSejdtcENJzmAVMXE
Routing:
- net (no net): track 121.0 -> 101.6 mm
Other:
- board text added: "1.0 .8"
- board text added: "1.0 .8 .5"
- board text added: "PCB MillBurn Test Board"
- board text added: "V 1.1"
- board text removed: "0.5"
- board text removed: "PCB MillBurn Test Board V1"
- board text removed: "V 1.0"

Commit message: Version 0.1.5: a board made with it, front and back
The whole mixed workflow ran on metal, 2026-09-20: 1.6 mm double-sided
clad, stock and its waste holes cut on the mill, both coppers burned
through paint and etched, drilled and cut out back on the mill with every
file corrected by the two-hole alignment measured from those waste holes,
then the mask openings and legend burned both sides. "The mask and
silkscreen alignment is perfect."

Three photographs of the finished board open the status section, stripped
of their camera metadata. Alignment from the stock's waste holes and the
placing layers leave the "not yet on metal" list, which is now down to
three items.

The test board's Gerbers come with it: the legend was redrawn in KiCad
during the run, so the corpus and the KiCad source are re-exported, and
the one test that pins the legend's imported size moves 64.01 to 64.06.

Co-Authored-By: Claude Opus 5 <noreply@anthropic.com>
Changed lines of the file:
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@@
+		)
+	)
+	(gr_text "1.0 .8 .5"
+		(at 174.0318 120.624 90)
+		(layer "F.SilkS")
+		(effects
+			(font
+				(size 1.5 1.5)
+				(thickness 0.3)
+				(bold yes)
+			)
+			(justify left bottom)
+		)
+	)
+	(gr_text "1.0 .8"
+		(at 174.147 128.524 90)
+		(layer "F.SilkS")
+		(effects
+			(font
+				(size 1.5 1.5)
+				(thickness 0.3)
+				(bold yes)
+			)
+			(justify left bottom)
+		)
+	)
+	(gr_text ".5    .8    1.0"
+		(at 150.097 143.841 0)
+		(layer "F.SilkS")
+		(effects
+			(font
+				(size 2 2)
+				(thickness 0.4)
+				(bold yes)
+			)
+			(justify left bottom)
+		)
+	)
+	(gr_text "V 1.1"
+		(at 180.3402 123.1882 90)
+		(layer "F.SilkS")
+		(effects
+			(font
+				(size 2 2)
+				(thickness 0.5)
+				(bold yes)
+			)
+			(justify left bottom)
+		)
+	)
+	(gr_text "MillBurn"
+		(at 180.3402 137.1582 90)
+		(layer "F.SilkS")
+		(effects
+			(font
+				(size 2 2)
+				(thickness 0.5)
+				(bold yes)
+			)
+			(justify left bottom)
 		)
 	)
@@
 			)
 		)
+	)
+	(zone
+		(layer "F.SilkS")
+		(hatch none 0.5)
+		(connect_pads
+			(clearance 0.5)
+		)
+		(min_thickness 0.25)
+		(fill yes
+			(thermal_gap 0.5)
+			(thermal_bridge_width 0.5)
+			(smoothing chamfer)
+			(radius 1)
+			(island_removal_mode 0)
+		)
+		(polygon
+			(pts
+				(xy 148.519083 129.840825) (xy 175.019425 129.84) (xy 175.019535 140.839736) (xy 148.519425 140.84)
+			)
+		)
